File: hardware/Starbiew.kicad_sch (KiCad schematic)
At the start: 23 parts, among them J1 Conn_01x04_Pin, J2 Conn_01x08_Pin, J3 MOTOR, Q1 AO3400A, SW1 SW_Push, SW2 SW_Push, U1 XIAO-ESP32-C3-SMD, U2 DHT11

Commit message: Prepare Starbie hardware package for submission.
🤖 Generated with Codebuff
Co-Authored-By: Codebuff <noreply@codebuff.com>
Connections:
- net +3.3V: now also D3.1 (K); no longer D3.2 (A)
- net at J3.2 (Pin_2), Q1.3 (D): now also D3.2 (A); no longer D3.1 (K)
Other:
- moved on the sheet: D3
Changed lines of the file:
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@@
 	)
 	(junction
-		(at 168.91 99.06)
+		(at 170.18 69.85)
 		(diameter 0)
 		(color 0 0 0 0)
 	)
 	(junction
-		(at 154.94 52.07)
+		(at 170.18 72.39)
 		(diameter 0)
 		(color 0 0 0 0)
 	)
 	(junction
-		(at 172.72 69.85)
+		(at 168.91 99.06)
 		(diameter 0)
 		(color 0 0 0 0)
 	)
 	(junction
-		(at 179.07 55.88)
+		(at 154.94 52.07)
 		(diameter 0)
 		(color 0 0 0 0)
 	)
 	(junction
-		(at 113.03 139.7)
+		(at 172.72 69.85)
 		(diameter 0)
 		(color 0 0 0 0)
 	)
 	(junction
-		(at 170.18 72.39)
+		(at 179.07 55.88)
 		(diameter 0)
 		(color 0 0 0 0)
 	)
 	(junction
-		(at 179.07 63.5)
+		(at 113.03 139.7)
 		(diameter 0)
 		(color 0 0 0 0)
 	)
 	(junction
-		(at 158.75 91.44)
+		(at 179.07 63.5)
 		(diameter 0)
 		(color 0 0 0 0)
 	)
 	(junction
-		(at 170.18 69.85)
+		(at 158.75 91.44)
 		(diameter 0)
 		(color 0 0 0 0)
@@
 	(wire
 		(pts
-			(xy 147.32 60.96) (xy 147.32 63.5)
+			(xy 170.18 69.85) (xy 172.72 69.85)
 		)
 		(stroke
@@
 	(wire
 		(pts
-			(xy 101.6 120.65) (xy 110.49 120.65)
+			(xy 147.32 60.96) (xy 147.32 63.5)
 		)
 		(stroke
@@
 	(wire
 		(pts
-			(xy 95.25 96.52) (xy 100.33 96.52)
+			(xy 101.6 120.65) (xy 110.49 120.65)
 		)
 		(stroke
@@
 	(wire
 		(pts
-			(xy 156.21 99.06) (xy 168.91 99.06)
+			(xy 95.25 96.52) (xy 100.33 96.52)
 		)
 		(stroke
@@
 	(wire
 		(pts
-			(xy 156.21 66.04) (xy 170.18 66.04)
+			(xy 156.21 99.06) (xy 168.91 99.06)
 		)
 		(stroke
@@
 	(wire
 		(pts
+			(xy 156.21 66.04) (xy 170.18 66.04)
+		)
+		(stroke
+			(width 0)
+			(type default)
+		)
+	)
+	(wire
+		(pts
 			(xy 170.18 66.04) (xy 170.18 69.85)
 		)
@@
 	(wire
 		(pts
-			(xy 170.18 73.66) (xy 170.18 72.39)
+			(xy 161.29 144.78) (xy 161.29 147.32)
 		)
 		(stroke
@@
 	(wire
 		(pts
-			(xy 161.29 144.78) (xy 161.29 147.32)
+			(xy 137.16 68.58) (xy 137.16 78.74)
 		)
 		(stroke
@@
 	(wire
 		(pts
-			(xy 137.16 68.58) (xy 137.16 78.74)
+			(xy 99.06 130.81) (xy 99.06 148.59)
 		)
 		(stroke
@@
 	(wire
 		(pts
-			(xy 99.06 130.81) (xy 99.06 148.59)
+			(xy 154.94 62.23) (xy 154.94 60.96)
 		)
 		(stroke
@@
 	(wire
 		(pts
-			(xy 154.94 62.23) (xy 154.94 60.96)
+			(xy 95.25 81.28) (xy 100.33 81.28)
 		)
 		(stroke
@@
 	(wire
 		(pts
-			(xy 95.25 81.28) (xy 100.33 81.28)
+			(xy 135.89 68.58) (xy 137.16 68.58)
 		)
 		(stroke
@@
 	(wire
 		(pts
-			(xy 135.89 68.58) (xy 137.16 68.58)
+			(xy 110.49 139.7) (xy 113.03 139.7)
 		)
 		(stroke
@@
 	(wire
 		(pts
-			(xy 110.49 139.7) (xy 113.03 139.7)
+			(xy 170.18 73.66) (xy 170.18 72.39)
 		)
 		(stroke
@@
 	(wire
 		(pts
+			(xy 170.18 72.39) (xy 190.5 72.39)
+		)
+		(stroke
+			(width 0)
+			(type default)
+		)
+	)
+	(wire
+		(pts
 			(xy 168.91 99.06) (xy 172.72 99.06)
 		)
@@
 	(wire
 		(pts
-			(xy 170.18 72.39) (xy 190.5 72.39)
+			(xy 168.91 72.39) (xy 170.18 72.39)
 		)
 		(stroke
@@
 	(wire
 		(pts
-			(xy 156.21 73.66) (xy 170.18 73.66)
-		)
-		(stroke
-			(width 0)
-			(type default)
-		)
-	)
-	(wire
-		(pts
 			(xy 105.41 102.87) (xy 114.3 102.87)
 		)
@@
 	(wire
 		(pts
-			(xy 88.9 119.38) (xy 88.9 127)
+			(xy 156.21 73.66) (xy 170.18 73.66)
 		)
 		(stroke
@@
 	(wire
 		(pts
-			(xy 110.49 148.59) (xy 110.49 139.7)
+			(xy 88.9 119.38) (xy 88.9 127)
 		)
 		(stroke
@@
 	(wire
 		(pts
-			(xy 210.82 96.52) (xy 210.82 100.33)
+			(xy 110.49 148.59) (xy 110.49 139.7)
 		)
 		(stroke
@@
 	(wire
 		(pts
-			(xy 203.2 132.08) (xy 203.2 135.89)
+			(xy 210.82 96.52) (xy 210.82 100.33)
 		)
 		(stroke
@@
 	(wire
 		(pts
-			(xy 179.07 63.5) (xy 179.07 66.04)
+			(xy 203.2 132.08) (xy 203.2 135.89)
 		)
 		(stroke
@@
 	(wire
 		(pts
-			(xy 170.18 69.85) (xy 172.72 69.85)
+			(xy 179.07 63.5) (xy 179.07 66.04)
 		)
 		(stroke
@@
 	(wire
 		(pts
-			(xy 168.91 72.39) (xy 170.18 72.39)
-		)
-		(stroke
-			(width 0)
-			(type default)
-		)
-	)
-	(wire
-		(pts
 			(xy 93.98 119.38) (xy 93.98 129.54)
 		)
@@
 	(symbol
 		(lib_id "Diode:SS14")
-		(at 156.21 69.85 90)
+		(at 156.21 69.85 270)
 		(unit 1)
 		(body_style 1)
@@
 		(dnp no)
 		(property "Reference" "D3"
-			(at 151.638 68.58 90)
+			(at 160.782 71.12 90)
 			(show_name no)
 			(do_not_autoplace no)
@@
 		)
 		(property "Value" "SS14"
-			(at 149.352 71.374 90)
+			(at 163.068 68.326 90)
 			(show_name no)
 			(do_not_autoplace no)
@@
 		)
 		(property "Footprint" "Diode_SMD:D_SOD-123"
-			(at 160.655 69.85 0)
+			(at 151.765 69.85 0)
 			(hide yes)
 			(show_name no)
