File: hardware/Starbiew.kicad_pcb (KiCad board)
At the start: 2 copper layers, 104 x 93.5 mm, 24 parts, among them J1 Conn_01x04_Pin, J2 Conn_01x08_Pin, J3 MOTOR, Q1 AO3400A, SW1 SW_Push, SW2 SW_Push, U1 XIAO-ESP32-C3-SMD, U2 DHT11

Commit message: Update custom PCB, regenerate gerbers, and refresh BOM prices
The PCB was edited after the last export, so the Gerbers, drill, position
file and zip are regenerated from the current board. The BOM now uses the
best verified prices with vendor order quantities and line totals.

🤖 Generated with Codebuff
Co-Authored-By: Codebuff <noreply@codebuff.com>
Other:
- board size 104 x 93.5 mm -> 98 x 93.5 mm
